File: Kicad_Stuff/StmBoard/StmBoard.kicad_sch (KiCad schematic)
At the start: 2 parts, among them U1 STM32G031K8Tx, U2 LIS3DH

Commit message: quick commit
Parts:
- added C1: 0.1Uf, symbol Device:C
- added C2: 10uf, symbol Device:C
- added R1, R2, R3, R4, R5, R6, R7: 10K, symbol Device:R
- added SW1, SW2, SW3, SW4, SW5, SW6, SW7: SW_DIP_x01, symbol Switch:SW_DIP_x01
Connections:
- net SCL: now also U1.19 (PA9/NC), U2.4 (SCL/SPC); no longer U1.22 (PA11/PA9)
- net SDA: now also U1.21 (PA10/NC), U2.6 (SDA/SDI/SDO); no longer U1.23 (PA12/PA10)
- net +3.3V: now reaches U2.1 (VDD_IO)
- net +3.3V: now also U2.14 (VDD), U2.8 (CS), C1.1, C2.1, SW1.1, SW2.1, SW3.1, SW4.1, SW5.1, SW6.1, SW7.1
- net GND: now reaches U2.10 (GND), U2.12 (GND), U2.5 (GND)
- net GND: now also U2.7 (SDO/SA0), C1.2, C2.2, R1.2, R2.2, R3.2, R4.2, R5.2, R6.2, R7.2
- new net A0: R4.1, SW1.2
- new net A1: R1.1, SW2.2
- new net A2: R2.1, SW3.2
- new net A3: R3.1, SW4.2
- new net A4: R5.1, SW5.2
- new net A5: R6.1, SW6.2
- new net A6: R7.1, SW7.2
Other:
- moved on the sheet: U2

Commit message: quick commit
Parts:
- added C3, C4: 1uf, symbol Device:C
- added C5: 0.1uf, symbol Device:C
- added C6: 3.3uf, symbol Device:C
- added R10, R9: R, symbol Device:R
- added R8: 10K, symbol Device:R
- added SW8: SW_DIP_x01, Button_Switch_SMD:SW_Push_1P1T_NO_CK_KSC6xxJ, symbol Switch:SW_DIP_x01
- added U10: ~, symbol custom:PortB_PinOut
- added U3, U4: ~, Custom:I2C_th_4_pin, symbol custom:I2C_4_Pin_THT_PORT
- added U5: ~, symbol custom:ADC_3_th_conector
- added U6: ~, symbol custom:Serial_Conecter_th
- added U7: ~, symbol custom:power_2_th
- added U8: MIC5504-3.3YM5, Package_TO_SOT_SMD:SOT-23-5, symbol Regulator_Linear:MIC5504-3.3YM5
- added U9: L78L05_SO8, Package_SO:SOIC-8_3.9x4.9mm_P1.27mm, symbol Regulator_Linear:L78L05_SO8
- SW1, SW2, SW3, SW4, SW5, SW6, SW7: footprint (none) -> Button_Switch_SMD:SW_Push_1P1T_NO_CK_KSC6xxJ
Connections:
- net +3.3V: now also C4.1, R10.1, R9.1, SW8.1, U3.1 (VCC), U4.1 (VCC), U8.5 (VOUT)
- net A0: now also U1.7 (PA0)
- net A1: now also U1.8 (PA1)
- net A2: now also U1.11 (PA4)
- net A3: now also U1.12 (PA5)
- net A4: now also U1.23 (PA12/PA10)
- net A5: now also U1.22 (PA11/PA9)
- net A6: now also U1.13 (PA6)
- net GND: now also C3.2, C4.2, C5.2, C6.2, R8.2, U3.0 (GND), U4.0 (GND), U7.2 (GDN), U8.2 (GND), U9.2 (GND), U9.3 (GND), U9.6 (GND), U9.7 (GND)
- net SCL: now also R10.2, U3.2 (SCL), U4.2 (SCL)
- net SDA: now also R9.2, U3.3 (SDA), U4.3 (SDA)
- net at U2.11 (INT1): now also U1.24 (PA13)
- net at U2.13 (ADC3): now also U5.3 (ADC3)
- net at U2.15 (ADC2): now also U5.2 (ADC2)
- net at U2.16 (ADC1): now also U5.1 (ADC1)
- net at U2.9 (INT2): now also U1.25 (PA14)
- net at U1.1 (PB9): now also U10.9 (PB_9)
- net RX_UASART2_VCOM: now reaches U1.10 (PA3)
- net RX_UASART2_VCOM: now also U6.1 (Rx)
- net A7: now reaches U1.14 (PA7)
- net A7: now also R8.1, SW8.2
- net at U1.15 (PB0): now also U10.0 (PB_0)
- net at U1.16 (PB1): now also U10.1 (PB_1)
- net at U1.17 (PB2): now also U10.2 (PB_2)
- net at U1.27 (PB3): now also U10.3 (PB_3)
- net at U1.28 (PB4): now also U10.4 (PB_4)
- net at U1.29 (PB5): now also U10.5 (PB_5)
- net at U1.30 (PB6): now also U10.6 (PB_6)
- net at U1.31 (PB7): now also U10.7 (PB_7)
- net at U1.32 (PB8): now also U10.8 (PB_8)
- net TX_UASART2_VCOM: now reaches U1.9 (PA2)
- net TX_UASART2_VCOM: now also U6.2 (Tx)
- new net: C6.1, U7.1 (VCC), U9.8 (IN)
- new net VCC: C3.1, C5.1, U8.1 (VIN), U9.1 (OUT)
Other:
- company: (none) -> NAIT
- title: (none) -> STM32 Firsst Board

Commit message: quick commit
Parts:
- added C7, C8: 10pf, symbol Device:C
- added Y1: 32Khz LSE, symbol Device:Crystal
Connections:
- net GND: now also U1.5 (VSS), C7.1, C8.1
- net at U2.11 (INT1): now also U1.18 (PA8); no longer U1.24 (PA13)
- net at U2.9 (INT2): now also U1.26 (PA15); no longer U1.25 (PA14)
- net at U1.2 (PC14): now also C8.2, Y1.2
- net at U1.3 (PC15): now also C7.2, Y1.1
- net reset: now reaches U1.6 (PF2)
- new net SWCLK: U1.25 (PA14)
- new net SWDIO: U1.24 (PA13)

Commit message: quick commit
Parts:
- added C10, C11: 100nf, symbol Device:C
- added C9: 4.7uf, symbol Device:C
- added SW9: SW_DIP_x01, Button_Switch_SMD:SW_Push_1P1T_NO_CK_KSC6xxJ, symbol Switch:SW_DIP_x01
Connections:
- net +3.3V: now also U1.4 (VDD), C10.2, C9.2
- net GND: now also C10.1, C11.1, C9.1, SW9.2
- net reset: now also C11.2, SW9.1

Commit message: quick commit
Parts:
- added U11: ~, symbol custom:gndnPower
Connections:
- net +3.3V: now also U11.4 (3.3v)
- net GND: now also U11.1 (gnd), U11.2 (gnd)
- new net +5V: U11.3 (5v)
Changed lines of the file:
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@@
   (junction (at 35.56 165.1) (diameter 0) (color 0 0 0 0)
   )
+  (junction (at 97.79 120.65) (diameter 0) (color 0 0 0 0)
+  )
   (junction (at 243.84 50.8) (diameter 0) (color 0 0 0 0)
   )
@@
   (junction (at 105.41 25.4) (diameter 0) (color 0 0 0 0)
   )
+  (wire (pts (xy 90.17 120.65) (xy 97.79 120.65))
+    (stroke (width 0) (type default))
+  )
   (wire (pts (xy 270.51 50.8) (xy 281.94 50.8))
     (stroke (width 0) (type default))
@@
     (stroke (width 0) (type default))
   )
+  (wire (pts (xy 90.17 115.57) (xy 99.06 115.57))
+    (stroke (width 0) (type default))
+  )
   (wire (pts (xy 119.38 64.77) (xy 132.08 64.77))
     (stroke (width 0) (type default))
@@
     (stroke (width 0) (type default))
   )
+  (wire (pts (xy 90.17 118.11) (xy 97.79 118.11))
+    (stroke (width 0) (type default))
+  )
   (wire (pts (xy 220.98 114.3) (xy 191.77 114.3))
     (stroke (width 0) (type default))
@@
     (stroke (width 0) (type default))
   )
+  (wire (pts (xy 97.79 120.65) (xy 100.33 120.65))
+    (stroke (width 0) (type default))
+  )
   (wire (pts (xy 91.44 36.83) (xy 81.28 36.83))
     (stroke (width 0) (type default))
@@
     (stroke (width 0) (type default))
   )
+  (wire (pts (xy 97.79 118.11) (xy 97.79 120.65))
+    (stroke (width 0) (type default))
+  )
   (wire (pts (xy 19.05 125.73) (xy 19.05 142.24))
     (stroke (width 0) (type default))
@@
   )
   (wire (pts (xy 138.43 57.15) (xy 119.38 57.15))
+    (stroke (width 0) (type default))
+  )
+  (wire (pts (xy 90.17 113.03) (xy 99.06 113.03))
     (stroke (width 0) (type default))
   )
@@
     )
   )
+  (symbol (lib_id "power:+3.3V") (at 99.06 113.03 270) (unit 1)
+    (in_bom yes) (on_board yes) (dnp no) (fields_autoplaced)
+    (property "Reference" "#PWR032" (at 95.25 113.03 0)
+      (effects (font (size 1.27 1.27)) hide)
+    )
+    (property "Value" "+3.3V" (at 102.87 113.03 90)
+      (effects (font (size 1.27 1.27)) (justify left))
+    )
+    (property "Footprint" "" (at 99.06 113.03 0)
+      (effects (font (size 1.27 1.27)) hide)
+    )
+    (property "Datasheet" "" (at 99.06 113.03 0)
+      (effects (font (size 1.27 1.27)) hide)
+    )
+    (pin "1")
+    (instances
+      (project "StmBoard"
+        (path "/27842249-4d05-45e0-a285-5f644f3ee952"
+          (reference "#PWR032") (unit 1)
+        )
+      )
+    )
+  )
   (symbol (lib_id "custom:I2C_4_Pin_THT_PORT") (at 184.15 25.4 0) (unit 1)
     (in_bom no) (on_board yes) (dnp no) (fields_autoplaced)
@@
     )
   )
+  (symbol (lib_id "power:+5V") (at 99.06 115.57 270) (unit 1)
+    (in_bom yes) (on_board yes) (dnp no) (fields_autoplaced)
+    (property "Reference" "#PWR033" (at 95.25 115.57 0)
+      (effects (font (size 1.27 1.27)) hide)
+    )
+    (property "Value" "+5V" (at 102.87 115.57 90)
+      (effects (font (size 1.27 1.27)) (justify left))
+    )
+    (property "Footprint" "" (at 99.06 115.57 0)
+      (effects (font (size 1.27 1.27)) hide)
+    )
+    (property "Datasheet" "" (at 99.06 115.57 0)
+      (effects (font (size 1.27 1.27)) hide)
+    )
+    (pin "1")
+    (instances
+      (project "StmBoard"
+        (path "/27842249-4d05-45e0-a285-5f644f3ee952"
+          (reference "#PWR033") (unit 1)
+        )
+      )
+    )
+  )
   (symbol (lib_id "Device:C") (at 43.18 21.59 0) (unit 1)
     (in_bom yes) (on_board yes) (dnp no) (fields_autoplaced)
@@
         (path "/27842249-4d05-45e0-a285-5f644f3ee952"
           (reference "R9") (unit 1)
+        )
+      )
+    )
+  )
+  (symbol (lib_id "custom:gndnPower") (at 90.17 116.84 90) (unit 1)
+    (in_bom yes) (on_board yes) (dnp no) (fields_autoplaced)
+    (property "Reference" "U11" (at 88.9 109.22 90)
+      (effects (font (size 1.27 1.27)))
+    )
+    (property "Value" "~" (at 90.17 116.84 0)
+      (effects (font (size 1.27 1.27)))
+    )
+    (property "Footprint" "" (at 90.17 116.84 0)
+      (effects (font (size 1.27 1.27)) hide)
+    )
+    (property "Datasheet" "" (at 90.17 116.84 0)
+      (effects (font (size 1.27 1.27)) hide)
+    )
+    (pin "3")
+    (pin "2")
+    (pin "1")
+    (pin "4")
+    (instances
+      (project "StmBoard"
+        (path "/27842249-4d05-45e0-a285-5f644f3ee952"
+          (reference "U11") (unit 1)
         )
       )
@@
         )
       )
+    )
+  )
+  (symbol (lib_id "power:GND") (at 100.33 120.65 90) (unit 1)
+    (in_bom yes) (on_board yes) (dnp no) (fields_autoplaced)
+    (property "Reference" "#PWR031" (at 106.68 120.65 0)
+      (effects (font (size 1.27 1.27)) hide)
+    )
+    (property "Value" "GND" (at 104.14 120.65 90)
+      (effects (font (size 1.27 1.27)) (justify right))
+    )
+    (property "Footprint" "" (at 100.33 120.65 0)
+      (effects (font (size 1.27 1.27)) hide)
+    )
+    (property "Datasheet" "" (at 100.33 120.65 0)
+      (effects (font (size 1.27 1.27)) hide)
+    )
+    (pin "1")
+    (instances
+      (project "StmBoard"
+        (path "/27842249-4d05-45e0-a285-5f644f3ee952"
+          (reference "#PWR031") (unit 1)
+        )
+      )

Commit message: quick commit
Parts:
- added U12: ~, Connector_PinHeader_2.54mm:PinHeader_1x05_P2.54mm_Vertical, symbol custom:STM32_PROG
- C1, C10, C11, C2, C3, C4, C5, C6, C7, C8, C9: footprint (none) -> Capacitor_SMD:C_0805_2012Metric
- R1, R2, R3, R4, R5, R6, R7, R8: footprint (none) -> Resistor_SMD:R_0603_1608Metric
- R10, R9: value R -> 10k; footprint (none) -> Resistor_SMD:R_0603_1608Metric
- SW1, SW2, SW3, SW4, SW5, SW6, SW7, SW8, SW9: footprint Button_Switch_SMD:SW_Push_1P1T_NO_CK_KSC6xxJ -> Button_Switch_THT:SW_PUSH_6mm
- U10: footprint (none) -> Connector_PinSocket_2.54mm:PinSocket_1x10_P2.54mm_Vertical
- U11: footprint (none) -> Connector_PinHeader_2.54mm:PinHeader_1x04_P2.54mm_Vertical
- U3, U4: footprint Custom:I2C_th_4_pin -> Connector_PinHeader_2.54mm:PinHeader_1x04_P2.54mm_Vertical
- U5: footprint (none) -> Connector_PinHeader_2.54mm:PinHeader_1x03_P2.54mm_Vertical
- U6, U7: footprint (none) -> Connector_PinHeader_2.54mm:PinHeader_1x02_P2.54mm_Vertical
- Y1: footprint (none) -> Crystal:Crystal_SMD_3215-2Pin_3.2x1.5mm
Connections:
- net +5V is gone; now on net VCC: U11.3 (5v)
- net +3.3V: now also U3.2 (VCC), U4.2 (VCC); no longer U3.1 (VCC), U4.1 (VCC)
- net GND: now also U1.20 (PC6), U3.1 (GND), U4.1 (GND), U12. (VCC); no longer U3.0 (GND), U4.0 (GND)
- net SCL: now also U3.3 (SCL), U4.3 (SCL); no longer U3.2 (SCL), U4.2 (SCL)
- net SDA: now also U3.4 (SDA), U4.4 (SDA); no longer U3.3 (SDA), U4.3 (SDA)
- net SWCLK: now also U12. (VCC)
- net SWDIO: now also U12. (VCC)
- net VCC: now also U8.3 (EN), U12. (VCC)
- net reset: now also U12. (VCC)
Other:
- moved on the sheet: U6

Commit message: quick commit
Parts:
- added C12: 0.1uf, Capacitor_SMD:C_0805_2012Metric, symbol Device:C
- added J1: USB_B_Mini, Connector_USB:USB_Mini-B_Lumberg_2486_01_Horizontal, symbol Connector:USB_B_Mini
- added U13: MCP2221AxST, Package_SO:TSSOP-14_4.4x5mm_P0.65mm, symbol Interface_USB:MCP2221AxST
Connections:
- net +3.3V: now also C12.1, U13.1 (VDD), U13.11 (VUSB), U13.4 (~{RST})
- net GND: now also C12.2, J1.5 (GND), J1.6 (Shield), U13.14 (VSS), U13.2 (GP0), U13.3 (GP1), U13.7 (GP2), U13.8 (GP3)
- net RX_UASART2_VCOM: now also U13.6 (UTx)
- net SWCLK: now also U13.10 (SCL)
- net SWDIO: now also U13.9 (SDA)
- net TX_UASART2_VCOM: now also U13.5 (URx)
- net at C6.1, U7.1 (VCC), U9.8 (IN): now also J1.1 (VBUS)
- new net: J1.2 (D-), U13.12 (D-)
- new net: J1.3 (D+), U13.13 (D+)
Other:
- moved on the sheet: U12

Commit message: quick commit
Connections:
- net GND: now also U12.1 (GND); no longer U12. (VCC)
- net SWCLK: now also U12.4 (SWCLK); no longer U12. (VCC)
- net SWDIO: now also U12.5 (SWDIO); no longer U12. (VCC)
- net VCC: now also U12.2 (VCC); no longer U12. (VCC)
- net reset: now also U12.3 (Reset); no longer U12. (VCC)
- net at U1.15 (PB0): now also U10.10 (PB_0); no longer U10.0 (PB_0)
Changed lines of the file:
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@@
     (stroke (width 0) (type default))
   )
-  (wire (pts (xy 119.38 118.11) (xy 134.62 118.11))
+  (wire (pts (xy 119.38 118.11) (xy 137.16 118.11))
     (stroke (width 0) (type default))
   )
@@
     (stroke (width 0) (type default))
   )
-  (wire (pts (xy 119.38 121.92) (xy 134.62 121.92))
+  (wire (pts (xy 119.38 121.92) (xy 137.16 121.92))
     (stroke (width 0) (type default))
   )
@@
     (stroke (width 0) (type default))
   )
-  (wire (pts (xy 119.38 114.3) (xy 134.62 114.3))
+  (wire (pts (xy 119.38 114.3) (xy 137.16 114.3))
     (stroke (width 0) (type default))
   )
@@
     (stroke (width 0) (type default))
   )
-  (wire (pts (xy 128.27 110.49) (xy 134.62 110.49))
+  (wire (pts (xy 128.27 110.49) (xy 137.16 110.49))
     (stroke (width 0) (type default))
   )
@@
     (stroke (width 0) (type default))
   )
-  (wire (pts (xy 128.27 106.68) (xy 134.62 106.68))
+  (wire (pts (xy 128.27 106.68) (xy 137.16 106.68))
     (stroke (width 0) (type default))
   )
@@
     )
   )
-  (symbol (lib_id "custom:STM32_PROG") (at 134.62 111.76 270) (unit 1)
-    (in_bom yes) (on_board yes) (dnp no) (fields_autoplaced)
-    (property "Reference" "U12" (at 146.05 114.3 90)
-      (effects (font (size 1.27 1.27)) (justify left))
-    )
-    (property "Value" "~" (at 134.62 111.76 0)
-      (effects (font (size 1.27 1.27)))
-    )
-    (property "Footprint" "Connector_PinHeader_2.54mm:PinHeader_1x05_P2.54mm_Vertical" (at 134.62 111.76 0)
-      (effects (font (size 1.27 1.27)) hide)
-    )
-    (property "Datasheet" "" (at 134.62 111.76 0)
-      (effects (font (size 1.27 1.27)) hide)
-    )
-    (pin "")
-    (pin "")
-    (pin "")
-    (pin "")
-    (pin "")
+  (symbol (lib_id "custom:STM32_PROG") (at 137.16 111.76 270) (unit 1)
+    (in_bom yes) (on_board yes) (dnp no) (fields_autoplaced)
+    (property "Reference" "U12" (at 148.59 114.3 90)
+      (effects (font (size 1.27 1.27)) (justify left))
+    )
+    (property "Value" "~" (at 137.16 111.76 0)
+      (effects (font (size 1.27 1.27)))
+    )
+    (property "Footprint" "Connector_PinHeader_2.54mm:PinHeader_1x05_P2.54mm_Vertical" (at 137.16 111.76 0)
+      (effects (font (size 1.27 1.27)) hide)
+    )
+    (property "Datasheet" "" (at 137.16 111.76 0)
+      (effects (font (size 1.27 1.27)) hide)
+    )
+    (pin "2")
+    (pin "3")
+    (pin "5")
+    (pin "4")
+    (pin "1")
     (instances
       (project "StmBoard"
@@
     (pin "6")
     (pin "7")
-    (pin "0")
-    (pin "2")
-    (instances
+    (pin "10")
+    (pin "2")
+    (instances
