File: Kicad_Stuff/StmBoard/StmBoard.kicad_pcb (KiCad board)
At the start: 2 copper layers, 43 parts, among them SW1 SW_DIP_x01, SW2 SW_DIP_x01, SW3 SW_DIP_x01, SW4 SW_DIP_x01, SW5 SW_DIP_x01, SW6 SW_DIP_x01, SW7 SW_DIP_x01, SW8 SW_DIP_x01, SW9 SW_DIP_x01, U1 STM32G031K8Tx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

Commit message: quick commit
Parts:
- added C12: 0.1uf, Capacitor_SMD:C_0805_2012Metric, F.Cu at (100.3, 116.7)
- added J1: USB_B_Mini, Connector_USB:USB_Mini-B_Lumberg_2486_01_Horizontal, F.Cu at (80.7, 115.1)
- added U13: MCP2221AxST, Package_SO:TSSOP-14_4.4x5mm_P0.65mm, F.Cu at (92.8, 114.2)
- moved SW9 17.9 mm to (97.8, 131.9)
- moved U12 9.95 mm to (79.6, 87.0)
- moved U7 8.90 mm to (81.5, 106.7), turned to -90 degrees
- turned U6 to 90 degrees

Commit message: quick commit
Parts:
- moved SW9 57.0 mm to (77.4, 78.7)
- moved C11 51.7 mm to (89.3, 80.1)
- moved C5 43.5 mm to (87.8, 87.9), turned to 90 degrees
- moved C6 42.1 mm to (99.0, 87.8), turned to -90 degrees
- moved C4 35.0 mm to (90.4, 93.3), turned to 180 degrees
- moved R10 34.2 mm to (146.6, 87.5), turned to 180 degrees
- moved R9 30.5 mm to (146.6, 90.5), turned to 180 degrees
- moved C7 29.6 mm to (133.2, 91.1)
- moved C8 28.8 mm to (127.2, 91.0), turned to 180 degrees
- moved C3 27.6 mm to (90.5, 99.6), turned to 180 degrees
- moved U9 18.3 mm to (93.6, 88.6)
- moved U8 16.6 mm to (92.7, 96.9)
- moved C12 12.5 mm to (112.4, 113.3)
- moved U5 12.5 mm to (167.8, 105.1)
- moved U4 7.98 mm to (168.4, 84.3)
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Connections:
- U10 pad 10: (no net) -> Net-(U1-PB0)
- U12 pad 1: (no net) -> GND
- U12 pad 2: (no net) -> VCC
- U12 pad 3: (no net) -> /reset
- U12 pad 4: (no net) -> SWCLK
- U12 pad 5: (no net) -> SWDIO
Routing:
- net /A1: track 0.00 -> 10.1 mm
- net /A0: track 0.00 -> 9.69 mm
- net /A2: track 0.00 -> 9.64 mm
- net /A4: track 0.00 -> 9.58 mm
- net /A5: track 0.00 -> 9.44 mm
- net /A3: track 0.00 -> 9.25 mm
Other:
- board outline added: 103.6 x 50.6 mm
- copper layers 2 -> 4

Commit message: quick commit
Parts:
- moved C10 26.3 mm to (124.7, 98.6)
- moved C9 26.3 mm to (124.7, 95.6)
- moved C2 13.0 mm to (124.6, 106.8), turned to 180 degrees
- moved C12 12.3 mm to (100.1, 114.1)
- moved C1 12.2 mm to (124.6, 108.8), turned to 180 degrees
- moved C4 2.72 mm to (93.1, 93.6)
- moved U2 0.83 mm to (129.4, 107.8)
Changed lines of the file:
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@@
   )
   (footprint "Capacitor_SMD:C_0805_2012Metric" (layer "F.Cu")
-    (at 112.4 113.3)
+    (at 100.1 114.1)
     (descr "Capacitor SMD 0805 (2012 Metric), square (rectangular) end terminal, IPC_7351 nominal, (Body size source: IPC-SM-782 page 76, https://www.pcb-3d.com/wordpress/wp-content/uploads/ipc-sm-782a_amendment_1_and_2.pdf, https://docs.google.com/spreadsheets/d/1BsfQQcO9C6DZCsRaXUlFlo91Tg2WpOkGARC1WS5S8t0/edit?usp=sharing), generated with kicad-footprint-generator")
     (tags "capacitor")
@@
   )
   (footprint "Capacitor_SMD:C_0805_2012Metric" (layer "F.Cu")
-    (at 112.4 109.3)
+    (at 124.6 108.8 180)
     (descr "Capacitor SMD 0805 (2012 Metric), square (rectangular) end terminal, IPC_7351 nominal, (Body size source: IPC-SM-782 page 76, https://www.pcb-3d.com/wordpress/wp-content/uploads/ipc-sm-782a_amendment_1_and_2.pdf, https://docs.google.com/spreadsheets/d/1BsfQQcO9C6DZCsRaXUlFlo91Tg2WpOkGARC1WS5S8t0/edit?usp=sharing), generated with kicad-footprint-generator")
     (tags "capacitor")
@@
     (fp_line (start 1 0.625) (end -1 0.625)
       (stroke (width 0.1) (type solid)) (layer "F.Fab"))
-    (pad "1" smd roundrect (at -0.95 0) (size 1 1.45) (layers "F.Cu" "F.Paste" "F.Mask") (roundrect_rratio 0.25)
+    (pad "1" smd roundrect (at -0.95 0 180) (size 1 1.45) (layers "F.Cu" "F.Paste" "F.Mask") (roundrect_rratio 0.25)
       (net 1 "+3.3V") (pintype "passive"))
-    (pad "2" smd roundrect (at 0.95 0) (size 1 1.45) (layers "F.Cu" "F.Paste" "F.Mask") (roundrect_rratio 0.25)
+    (pad "2" smd roundrect (at 0.95 0 180) (size 1 1.45) (layers "F.Cu" "F.Paste" "F.Mask") (roundrect_rratio 0.25)
       (net 2 "GND") (pintype "passive"))
     (model "${KICAD6_3DMODEL_DIR}/Capacitor_SMD.3dshapes/C_0805_2012Metric.wrl"
@@
   )
   (footprint "Package_LGA:LGA-16_3x3mm_P0.5mm_LayoutBorder3x5y" (layer "F.Cu")
-    (at 128.6 107.5)
+    (at 129.375 107.8)
     (descr "LGA, 16 Pin (http://www.st.com/resource/en/datasheet/lis331hh.pdf), generated with kicad-footprint-generator ipc_noLead_generator.py")
     (tags "LGA NoLead")
@@
   )
   (footprint "Capacitor_SMD:C_0805_2012Metric" (layer "F.Cu")
-    (at 112.4 111.3)
+    (at 124.6 106.8 180)
     (descr "Capacitor SMD 0805 (2012 Metric), square (rectangular) end terminal, IPC_7351 nominal, (Body size source: IPC-SM-782 page 76, https://www.pcb-3d.com/wordpress/wp-content/uploads/ipc-sm-782a_amendment_1_and_2.pdf, https://docs.google.com/spreadsheets/d/1BsfQQcO9C6DZCsRaXUlFlo91Tg2WpOkGARC1WS5S8t0/edit?usp=sharing), generated with kicad-footprint-generator")
     (tags "capacitor")
@@
     (fp_line (start 1 0.625) (end -1 0.625)
       (stroke (width 0.1) (type solid)) (layer "F.Fab"))
-    (pad "1" smd roundrect (at -0.95 0) (size 1 1.45) (layers "F.Cu" "F.Paste" "F.Mask") (roundrect_rratio 0.25)
+    (pad "1" smd roundrect (at -0.95 0 180) (size 1 1.45) (layers "F.Cu" "F.Paste" "F.Mask") (roundrect_rratio 0.25)
       (net 1 "+3.3V") (pintype "passive"))
-    (pad "2" smd roundrect (at 0.95 0) (size 1 1.45) (layers "F.Cu" "F.Paste" "F.Mask") (roundrect_rratio 0.25)
+    (pad "2" smd roundrect (at 0.95 0 180) (size 1 1.45) (layers "F.Cu" "F.Paste" "F.Mask") (roundrect_rratio 0.25)
       (net 2 "GND") (pintype "passive"))
     (model "${KICAD6_3DMODEL_DIR}/Capacitor_SMD.3dshapes/C_0805_2012Metric.wrl"
@@
   )
   (footprint "Capacitor_SMD:C_0805_2012Metric" (layer "F.Cu")
-    (at 113.9 119.6)
+    (at 124.7 95.6)
     (descr "Capacitor SMD 0805 (2012 Metric), square (rectangular) end terminal, IPC_7351 nominal, (Body size source: IPC-SM-782 page 76, https://www.pcb-3d.com/wordpress/wp-content/uploads/ipc-sm-782a_amendment_1_and_2.pdf, https://docs.google.com/spreadsheets/d/1BsfQQcO9C6DZCsRaXUlFlo91Tg2WpOkGARC1WS5S8t0/edit?usp=sharing), generated with kicad-footprint-generator")
     (tags "capacitor")
@@
   )
   (footprint "Capacitor_SMD:C_0805_2012Metric" (layer "F.Cu")
-    (at 90.4 93.3 180)
+    (at 93.1 93.6 180)
     (descr "Capacitor SMD 0805 (2012 Metric), square (rectangular) end terminal, IPC_7351 nominal, (Body size source: IPC-SM-782 page 76, https://www.pcb-3d.com/wordpress/wp-content/uploads/ipc-sm-782a_amendment_1_and_2.pdf, https://docs.google.com/spreadsheets/d/1BsfQQcO9C6DZCsRaXUlFlo91Tg2WpOkGARC1WS5S8t0/edit?usp=sharing), generated with kicad-footprint-generator")
     (tags "capacitor")
@@
   )
   (footprint "Capacitor_SMD:C_0805_2012Metric" (layer "F.Cu")
-    (at 113.9 122.61)
+    (at 124.7 98.61)
     (descr "Capacitor SMD 0805 (2012 Metric), square (rectangular) end terminal, IPC_7351 nominal, (Body size source: IPC-SM-782 page 76, https://www.pcb-3d.com/wordpress/wp-content/uploads/ipc-sm-782a_amendment_1_and_2.pdf, https://docs.google.com/spreadsheets/d/1BsfQQcO9C6DZCsRaXUlFlo91Tg2WpOkGARC1WS5S8t0/edit?usp=sharing), generated with kicad-footprint-generator")
     (tags "capacitor")

Commit message: quick commit
Parts:
- moved U10 37.4 mm to (154.3, 80.3), turned to -90 degrees
- moved U11 27.5 mm to (117.2, 80.1)
- moved C10 6.06 mm to (130.1, 101.3)
- moved C8 5.93 mm to (133.1, 91.6)
- moved C1 5.87 mm to (119.2, 111.1)
- moved C9 5.24 mm to (128.4, 99.3)
- moved C7 4.83 mm to (128.4, 91.6)
- moved J1 2.05 mm to (79.5, 115.0)
- moved C2 1.24 mm to (125.8, 106.8)
- moved C11 0.83 mm to (88.6, 79.8), turned to 90 degrees
- moved SW9 0.77 mm to (78.2, 78.6)
- moved U12 0.74 mm to (78.3, 88.2)
- turned C5 to -90 degrees
- turned Y1 to 180 degrees
Connections:
- J1 pad 4: unconnected-(J1-ID-Pad4) -> GND
- U13 pad 10: SWCLK -> /SCL
- U13 pad 9: SWDIO -> /SDA
Routing:
- net /SDA: track 0.00 -> 164.4 mm, vias 0 -> 6
- net /SCL: track 0.00 -> 157.1 mm, vias 0 -> 6
- net /A0: track 9.69 -> 143.1 mm, vias 0 -> 1
- net /A7: track 0.00 -> 116.7 mm, vias 0 -> 4
- net GND: track 0.00 -> 112.7 mm, vias 0 -> 19
- net Net-(U1-PB0): track 0.00 -> 99.3 mm, vias 0 -> 3
- net VCC: track 0.00 -> 96.5 mm, vias 0 -> 3
- net Net-(U1-PB1): track 0.00 -> 94.3 mm, vias 0 -> 1
- net /A5: track 9.44 -> 103.1 mm, vias 0 -> 2
- net /reset: track 0.00 -> 93.3 mm, vias 0 -> 2
- net Net-(U1-PB2): track 0.00 -> 82.8 mm
- net /RX_UASART2_VCOM: track 0.00 -> 78.8 mm, vias 0 -> 1
- net /TX_UASART2_VCOM: track 0.00 -> 78.1 mm, vias 0 -> 3
- net /A4: track 9.58 -> 84.0 mm, vias 0 -> 1
- net SWDIO: track 0.00 -> 71.3 mm, vias 0 -> 1
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- added copper zone on In2.Cu, net +3.3V
- added copper zone on F.Cu, net GND
- added copper zone on In1.Cu, net GND
Other:
- board size 103.6 x 50.6 mm -> 106.1 x 53 mm
- board text added: "2024"
- board text added: "stm32G0 Micro B.Carpenter Nait"
